File: 8x8_eyes.kicad_sch (KiCad schematic)
At the start: 13 parts, among them J1 Conn_01x05_Female, U1 74HC595, U2 74HC595

Commit message: fix
Parts:
- J1: footprint Connector_Wago:Wago_734-135_1x05_P3.50mm_Vertical -> Connector_Molex:Molex_KK-254_AE-6410-05A_1x05_P2.54mm_Vertical
- U1, U2: footprint Package_SO:SOIC-16W_5.3x10.2mm_P1.27mm -> Package_DIP:DIP-16_W7.62mm
Connections:
- net CLR: now also J1.4 (Pin_4); no longer J1.1 (Pin_1)
- net GND: now also J1.1 (Pin_1); no longer J1.4 (Pin_4)
Changed lines of the file:
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@@
-    (stroke (width 0) (type default) (color 0 0 0 0))
-  )
-  (wire (pts (xy 43.18 107.95) (xy 46.99 107.95))
     (stroke (width 0) (type default) (color 0 0 0 0))
   )
@@
     (stroke (width 0) (type default) (color 0 0 0 0))
   )
+  (wire (pts (xy 43.18 100.33) (xy 54.102 100.33))
+    (stroke (width 0) (type default) (color 0 0 0 0))
+  )
   (wire (pts (xy 121.92 40.64) (xy 134.62 40.64))
     (stroke (width 0) (type default) (color 0 0 0 0))
@@
     )
   )
-  (global_label "CLR" (shape output) (at 46.99 107.95 0) (fields_autoplaced)
-    (effects (font (size 1.27 1.27)) (justify left))
-    (property "Intersheet References" "${INTERSHEET_REFS}" (id 0) (at 52.9712 108.0294 0)
+  (global_label "CLR" (shape output) (at 54.102 100.33 0) (fields_autoplaced)
+    (effects (font (size 1.27 1.27)) (justify left))
+    (property "Intersheet References" "${INTERSHEET_REFS}" (id 0) (at 60.0832 100.4094 0)
       (effects (font (size 1.27 1.27)) (justify left) hide)
     )
@@
     (in_bom yes) (on_board yes)
     (property "Reference" "R5" (id 0) (at 146.05 87.63 0)
-      (effects (font (size 1.27 1.27)) (justify left))
+      (effects (font (size 1.27 1.27)) (justify left) hide)
     )
     (property "Value" "220" (id 1) (at 147.32 90.17 0)
-      (effects (font (size 1.27 1.27)) (justify left))
+      (effects (font (size 1.27 1.27)) (justify left) hide)
     )
     (property "Footprint" "Resistor_THT:R_Axial_DIN0204_L3.6mm_D1.6mm_P5.08mm_Horizontal" (id 2) (at 145.542 90.17 90)
@@
     (in_bom yes) (on_board yes)
     (property "Reference" "R1" (id 0) (at 138.43 90.17 0)
-      (effects (font (size 1.27 1.27)) (justify left))
+      (effects (font (size 1.27 1.27)) (justify left) hide)
     )
     (property "Value" "220" (id 1) (at 138.43 92.71 0)
-      (effects (font (size 1.27 1.27)) (justify left))
+      (effects (font (size 1.27 1.27)) (justify left) hide)
     )
     (property "Footprint" "Resistor_THT:R_Axial_DIN0204_L3.6mm_D1.6mm_P5.08mm_Horizontal" (id 2) (at 137.922 91.44 90)
@@
     (property "Reference" "J1" (id 0) (at 38.735 92.71 0))
     (property "Value" "Conn_01x05_Female" (id 1) (at 38.735 95.25 0))
-    (property "Footprint" "Connector_Wago:Wago_734-135_1x05_P3.50mm_Vertical" (id 2) (at 38.1 102.87 0)
+    (property "Footprint" "Connector_Molex:Molex_KK-254_AE-6410-05A_1x05_P2.54mm_Vertical" (id 2) (at 38.1 102.87 0)
       (effects (font (size 1.27 1.27)) hide)
     )
@@
       (effects (font (size 1.27 1.27)) (justify left))
     )
-    (property "Footprint" "Package_SO:SOIC-16W_5.3x10.2mm_P1.27mm" (id 2) (at 44.45 48.26 0)
+    (property "Footprint" "Package_DIP:DIP-16_W7.62mm" (id 2) (at 44.45 48.26 0)
       (effects (font (size 1.27 1.27)) hide)
     )
@@
     (in_bom yes) (on_board yes) (fields_autoplaced)
     (property "Reference" "R3" (id 0) (at 147.32 132.0799 0)
-      (effects (font (size 1.27 1.27)) (justify left))
-    )
-    (property "Value" "220" (id 1) (at 147.32 134.6199 0)
-      (effects (font (size 1.27 1.27)) (justify left))
+      (effects (font (size 1.27 1.27)) (justify left) hide)
+    )
+    (property "Value" "220" (id 1) (at 147.32 133.3499 0)
+      (effects (font (size 1.27 1.27)) (justify left) hide)
     )
     (property "Footprint" "Resistor_THT:R_Axial_DIN0204_L3.6mm_D1.6mm_P5.08mm_Horizontal" (id 2) (at 143.002 133.35 90)
@@
     (in_bom yes) (on_board yes)
     (property "Reference" "R7" (id 0) (at 134.62 88.9 0)
-      (effects (font (size 1.27 1.27)) (justify left))
+      (effects (font (size 1.27 1.27)) (justify left) hide)
     )
     (property "Value" "220" (id 1) (at 133.35 95.25 0)
-      (effects (font (size 1.27 1.27)) (justify left))
+      (effects (font (size 1.27 1.27)) (justify left) hide)
     )
     (property "Footprint" "Resistor_THT:R_Axial_DIN0204_L3.6mm_D1.6mm_P5.08mm_Horizontal" (id 2) (at 132.842 90.17 90)
@@
     (in_bom yes) (on_board yes)
     (property "Reference" "R6" (id 0) (at 143.51 90.17 0)
-      (effects (font (size 1.27 1.27)) (justify left))
+      (effects (font (size 1.27 1.27)) (justify left) hide)
     )
     (property "Value" "220" (id 1) (at 142.24 91.44 0)
-      (effects (font (size 1.27 1.27)) (justify left))
+      (effects (font (size 1.27 1.27)) (justify left) hide)
     )
     (property "Footprint" "Resistor_THT:R_Axial_DIN0204_L3.6mm_D1.6mm_P5.08mm_Horizontal" (id 2) (at 143.002 90.17 90)
@@
     (in_bom yes) (on_board yes)
     (property "Reference" "R4" (id 0) (at 142.24 128.2699 0)
-      (effects (font (size 1.27 1.27)) (justify left))
+      (effects (font (size 1.27 1.27)) (justify left) hide)
     )
     (property "Value" "220" (id 1) (at 142.24 130.8099 0)
-      (effects (font (size 1.27 1.27)) (justify left))
+      (effects (font (size 1.27 1.27)) (justify left) hide)
     )
     (property "Footprint" "Resistor_THT:R_Axial_DIN0204_L3.6mm_D1.6mm_P5.08mm_Horizontal" (id 2) (at 137.922 129.54 90)
@@
     (in_bom yes) (on_board yes)
     (property "Reference" "R2" (id 0) (at 139.7 134.6199 0)
-      (effects (font (size 1.27 1.27)) (justify left))
+      (effects (font (size 1.27 1.27)) (justify left) hide)
     )
     (property "Value" "220" (id 1) (at 139.7 137.1599 0)
-      (effects (font (size 1.27 1.27)) (justify left))
+      (effects (font (size 1.27 1.27)) (justify left) hide)
     )
     (property "Footprint" "Resistor_THT:R_Axial_DIN0204_L3.6mm_D1.6mm_P5.08mm_Horizontal" (id 2) (at 135.382 135.89 90)
@@
       (effects (font (size 1.27 1.27)) (justify left))
     )
-    (property "Footprint" "Package_SO:SOIC-16W_5.3x10.2mm_P1.27mm" (id 2) (at 111.76 48.26 0)
+    (property "Footprint" "Package_DIP:DIP-16_W7.62mm" (id 2) (at 111.76 48.26 0)
       (effects (font (size 1.27 1.27)) hide)
     )
@@
     (pin "1")
   )
-  (symbol (lib_id "power:GND") (at 43.18 100.33 90) (unit 1)
-    (in_bom yes) (on_board yes) (fields_autoplaced)
-    (property "Reference" "#PWR0107" (id 0) (at 49.53 100.33 0)
-      (effects (font (size 1.27 1.27)) hide)
-    )
-    (property "Value" "GND" (id 1) (at 46.99 100.3299 90)
+  (symbol (lib_id "power:GND") (at 43.18 107.95 90) (unit 1)
+    (in_bom yes) (on_board yes)
+    (property "Reference" "#PWR0107" (id 0) (at 49.53 107.95 0)
+      (effects (font (size 1.27 1.27)) hide)
+    )
+    (property "Value" "GND" (id 1) (at 58.928 129.032 90)
       (effects (font (size 1.27 1.27)) (justify right))
     )
-    (property "Footprint" "" (id 2) (at 43.18 100.33 0)
-      (effects (font (size 1.27 1.27)) hide)
-    )
-    (property "Datasheet" "" (id 3) (at 43.18 100.33 0)
+    (property "Footprint" "" (id 2) (at 43.18 107.95 0)
+      (effects (font (size 1.27 1.27)) hide)
+    )
+    (property "Datasheet" "" (id 3) (at 43.18 107.95 0)
       (effects (font (size 1.27 1.27)) hide)
     )
@@
     )
     (path "/23f78ecd-ef55-49a3-b594-a4a6fd1a0ef1"
-      (reference "J1") (unit 1) (value "Conn_01x05_Female") (footprint "Connector_Wago:Wago_734-135_1x05_P3.50mm_Vertical")
+      (reference "J1") (unit 1) (value "Conn_01x05_Female") (footprint "Connector_Molex:Molex_KK-254_AE-6410-05A_1x05_P2.54mm_Vertical")
     )
     (path "/208d3c3f-1bea-4376-a2a1-c49062cdb734"
@@
     )
     (path "/322f1cc8-4c02-4383-a052-42ffb4923626"
-      (reference "U1") (unit 1) (value "74HC595") (footprint "Package_SO:SOIC-16W_5.3x10.2mm_P1.27mm")
+      (reference "U1") (unit 1) (value "74HC595") (footprint "Package_DIP:DIP-16_W7.62mm")
     )
     (path "/b121b379-3660-4945-a964-c9de59d50e9b"
-      (reference "U2") (unit 1) (value "74HC595") (footprint "Package_SO:SOIC-16W_5.3x10.2mm_P1.27mm")
-    )
-  )
+      (reference "U2") (unit 1) (value "74HC595") (footprint "Package_DIP:DIP-16_W7.62mm")
+    )
+  )

Commit message: fix
Connections:
- net +5V: now also J1.1 (Pin_1); no longer J1.5 (Pin_5)
- net GND: now also J1.5 (Pin_5); no longer J1.1 (Pin_1)
Changed lines of the file:
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@@
-    (stroke (width 0) (type default) (color 0 0 0 0))
-  )
-  (wire (pts (xy 43.18 97.79) (xy 46.99 97.79))
     (stroke (width 0) (type default) (color 0 0 0 0))
   )
@@
     )
   )
-  (global_label "VCC" (shape output) (at 46.99 97.79 0) (fields_autoplaced)
-    (effects (font (size 1.27 1.27)) (justify left))
-    (property "Intersheet References" "${INTERSHEET_REFS}" (id 0) (at 53.0317 97.7106 0)
+  (global_label "VCC" (shape output) (at 43.18 107.95 0) (fields_autoplaced)
+    (effects (font (size 1.27 1.27)) (justify left))
+    (property "Intersheet References" "${INTERSHEET_REFS}" (id 0) (at 49.2217 107.8706 0)
       (effects (font (size 1.27 1.27)) (justify left) hide)
     )
@@
     (pin "1")
   )
+  (symbol (lib_id "power:GND") (at 43.18 97.79 90) (unit 1)
+    (in_bom yes) (on_board yes) (fields_autoplaced)
+    (property "Reference" "#PWR0107" (id 0) (at 49.53 97.79 0)
+      (effects (font (size 1.27 1.27)) hide)
+    )
+    (property "Value" "GND" (id 1) (at 46.99 97.7899 90)
+      (effects (font (size 1.27 1.27)) (justify right))
+    )
+    (property "Footprint" "" (id 2) (at 43.18 97.79 0)
+      (effects (font (size 1.27 1.27)) hide)
+    )
+    (property "Datasheet" "" (id 3) (at 43.18 97.79 0)
+      (effects (font (size 1.27 1.27)) hide)
+    )
+    (pin "1")
+  )
   (symbol (lib_id "Device:R") (at 137.16 135.89 0) (unit 1)
     (in_bom yes) (on_board yes)
@@
     (pin "1")
   )
-  (symbol (lib_id "power:GND") (at 43.18 107.95 90) (unit 1)
-    (in_bom yes) (on_board yes)
-    (property "Reference" "#PWR0107" (id 0) (at 49.53 107.95 0)
-      (effects (font (size 1.27 1.27)) hide)
-    )
-    (property "Value" "GND" (id 1) (at 58.928 129.032 90)
-      (effects (font (size 1.27 1.27)) (justify right))
-    )
-    (property "Footprint" "" (id 2) (at 43.18 107.95 0)
-      (effects (font (size 1.27 1.27)) hide)
-    )
-    (property "Datasheet" "" (id 3) (at 43.18 107.95 0)
-      (effects (font (size 1.27 1.27)) hide)
-    )
-    (pin "1")
-  )
   (symbol (lib_id "power:+5V") (at 228.6 154.94 0) (unit 1)
     (in_bom yes) (on_board yes) (fields_autoplaced)
@@
       (reference "#PWR0106") (unit 1) (value "GND") (footprint "")
     )
-    (path "/c9618272-9fca-4bee-8a3d-1660fb195be2"
+    (path "/58a5a6aa-4ac1-454e-99de-9b74e53d0180"
       (reference "#PWR0107") (unit 1) (value "GND") (footprint "")
     )
