File: 8x8_eyes.kicad_pcb (KiCad board)
At the start: 2 copper layers, 13 parts, among them J1 Conn_01x05_Female, U1 74HC595, U2 74HC595

Commit message: add
Routing:
- net VCC: track 0.00 -> 81.3 mm
- net Pin 3: track 0.00 -> 62.2 mm, vias 0 -> 1
- net GND: track 0.00 -> 60.1 mm, vias 0 -> 11
- net Pin 4: track 0.00 -> 55.8 mm, vias 0 -> 1
- net Pin 6: track 0.00 -> 50.9 mm, vias 0 -> 1
- net CLK: track 0.00 -> 47.8 mm
- net Pin 16: track 0.00 -> 40.9 mm
- net Pin 1: track 0.00 -> 37.8 mm
- net Pin 2: track 0.00 -> 34.2 mm
- net Pin 13: track 0.00 -> 34.2 mm
- net Pin 12: track 0.00 -> 34.2 mm
- net Pin 15: track 0.00 -> 33.4 mm
- net Pin 14: track 0.00 -> 32.3 mm
- net Pin 8: track 0.00 -> 32.1 mm, vias 0 -> 1
- net CLR: track 0.00 -> 30.5 mm
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- added copper zone on B.Cu, net GND
- added copper zone on F.Cu, net GND
Other:
- board outline added: 71.1 x 63.5 mm

Commit message: fix
Parts:
- C1: moved to B.Cu
- J1: footprint Connector_Wago:Wago_734-135_1x05_P3.50mm_Vertical -> Connector_Molex:Molex_KK-254_AE-6410-05A_1x05_P2.54mm_Vertical; moved to B.Cu
- U1, U2: footprint Package_SO:SOIC-16W_5.3x10.2mm_P1.27mm -> Package_DIP:DIP-16_W7.62mm
- moved C1 18.3 mm to (149.9, 115.5)
- moved R2 17.8 mm to (134.6, 106.7)
- moved R3 17.8 mm to (142.2, 106.7)
- moved R4 17.8 mm to (137.2, 111.8)
- moved R1 15.2 mm to (137.2, 96.5)
- moved R5 15.2 mm to (144.8, 96.5)
- moved R6 15.2 mm to (142.2, 96.5)
- moved R7 15.2 mm to (132.1, 96.5)
- moved R8 15.2 mm to (129.5, 91.4)
- moved J1 13.6 mm to (165.1, 127.0), turned to 180 degrees
- moved U2 10.9 mm to (158.8, 80.0)
- moved U1 6.46 mm to (158.8, 102.9)
Connections:
- J1 pad 1: CLR -> GND
- J1 pad 4: GND -> CLR
Routing:
- net Pin 4: track 55.8 -> 33.9 mm, vias 1 -> 0
- net Pin 9: track 27.3 -> 49.0 mm
- net Pin 12: track 34.2 -> 54.4 mm
- net Pin 6: track 50.9 -> 31.1 mm, vias 1 -> 0
- net Pin 3: track 62.2 -> 42.7 mm, vias 1 -> 0
- net GND: track 60.1 -> 76.0 mm, vias 11 -> 7
- net CLR: track 30.5 -> 46.1 mm
- net Pin 14: track 32.3 -> 45.6 mm
- net CASCADE: track 25.3 -> 38.0 mm
- net Pin 7: track 26.0 -> 15.9 mm
- net Net-(D65-Pad4): track 13.8 -> 4.79 mm
- net Net-(D65-Pad10): track 12.3 -> 3.80 mm
- net Net-(D65-Pad15): track 12.3 -> 3.80 mm
- net Net-(D65-Pad11): track 12.3 -> 3.80 mm
- net Net-(D65-Pad13): track 12.3 -> 3.80 mm
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Other:
- board size 71.1 x 63.5 mm -> 55.9 x 58.4 mm
- board text added: "1"
- board text added: "2"
- board text added: "3"
- board text added: "4"
- board text added: "5"
- board text added: "CLK"
- board text added: "CLR"
- board text added: "GND"
- board text added: "K.Tanaka"
- board text added: "SER"
- board text added: "VCC"

Commit message: fix
Parts:
- added G***: LOGO, LOGO, F.Cu at (124.5, 127.0)
- moved C1 2.54 mm to (152.4, 115.5)
- moved R2 2.54 mm to (132.1, 106.7)
- moved R5 2.54 mm to (147.3, 96.5)
- moved R8 2.54 mm to (127.0, 91.4)
Connections:
- J1 pad 1: GND -> VCC
- J1 pad 5: VCC -> GND
Routing:
- net Pin 12: track 54.4 -> 30.0 mm, vias 0 -> 1
- net Pin 8: track 35.3 -> 16.5 mm
- net GND: track 76.0 -> 62.1 mm, vias 7 -> 6
- net Pin 9: track 49.0 -> 35.9 mm
- net Pin 14: track 45.6 -> 32.6 mm, vias 0 -> 1
- net VCC: track 73.7 -> 83.1 mm
- net Pin 13: track 35.0 -> 41.3 mm
- net Pin 11: track 19.1 -> 24.0 mm, vias 0 -> 1
- net CLR: track 46.1 -> 41.9 mm
- net Pin 3: track 42.7 -> 46.3 mm
- net CLK: track 48.3 -> 46.3 mm
- net Pin 10: track 18.7 -> 16.8 mm
- net Pin 2: track 35.0 -> 33.5 mm
- net Pin 16: track 35.5 -> 36.9 mm
- net Net-(D65-Pad10): track 3.80 -> 5.13 mm
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Other:
- board text added: "8x8 eyes"
- board text added: "Kengo Tanaka Presents"
- board text removed: "K.Tanaka"

Commit message: fix
Parts:
- removed G***: LOGO, LOGO
- added REF**: MountingHole_2.1mm, MountingHole:MountingHole_2.1mm, F.Cu at (149.9, 81.3)
- added REF**: MountingHole_2.1mm, MountingHole:MountingHole_2.1mm, F.Cu at (149.9, 129.5)
- added REF**: MountingHole_2.1mm, MountingHole:MountingHole_2.1mm, F.Cu at (119.4, 129.5)
- added REF**: MountingHole_2.1mm, MountingHole:MountingHole_2.1mm, F.Cu at (119.4, 81.3)
Other:
- board text removed: "Kengo Tanaka Presents"
